File: GW28R8128.sch (KiCad schematic (older format))
At the start: 8 parts, among them J1 Socket, U1 39SF010

Commit message: Revert "Forked header, as submitted to JLCPCB"
This reverts commit d1e7a343920c14c85af64a4568f625ea3f5c50c3.
Parts:
- removed J1: Socket, stdpads:DIP-28_W15.24mm_Socket_Inverse_Forked, symbol Connector_Generic:Conn_02x14_Counter_Clockwise
- added J1: Left, Connector_PinHeader_2.54mm:PinHeader_1x14_P2.54mm_Vertical, symbol Connector:Conn_01x14_Male
- added J2: Right, Connector_PinHeader_2.54mm:PinHeader_1x14_P2.54mm_Vertical, symbol Connector:Conn_01x14_Male
- U1: symbol GW_RAM:Flash-512Kx8-PLCC-32 -> stdparts:39F040
Connections:
- net +5V: now also J2.1 (Pin_1)
- net A0: now also J1.10 (Pin_10)
- net A1: now also J1.9 (Pin_9)
- net A10: now also J2.8 (Pin_8)
- net A11: now also J2.6 (Pin_6)
- net A12: now also J1.2 (Pin_2)
- net A13: now also J2.3 (Pin_3)
- net A14: now also J2.2 (Pin_2)
- net A15: now also J1.1 (Pin_1)
- net A16: now also J2.7 (Pin_7)
- net A2: now also J1.8 (Pin_8)
- net A3: now also J1.7 (Pin_7)
- net A4: now also J1.6 (Pin_6)
- net A5: now also J1.5 (Pin_5)
- net A6: now also J1.4 (Pin_4)
- net A7: now also J1.3 (Pin_3)
- net A8: now also J2.4 (Pin_4)
- net A9: now also J2.5 (Pin_5)
- net D0: now also J1.11 (Pin_11)
- net D1: now also J1.12 (Pin_12)
- net D2: now also J1.13 (Pin_13)
- net D3: now also J2.14 (Pin_14)
- net D4: now also J2.13 (Pin_13)
- net D5: now also J2.12 (Pin_12)
- net D6: now also J2.11 (Pin_11)
- net D7: now also J2.10 (Pin_10)
- net GND: now also J1.14 (Pin_14)
- net ~CS~: now also J2.9 (Pin_9)
Changed lines of the file:
@@
 	1    0    0    -1
 $EndComp
-Text Label 2300 3150 2    50   ~ 0
+$Comp
+L stdparts:39F040 U1
+U 1 1 5E56BC07
+P 2700 2450
+F 0 "U1" H 2700 3500 50  0000 C CNN
+F 1 "39SF010" V 2700 2450 50  0000 C CNN
+F 2 "stdpads:PLCC-32" H 2700 2450 50  0001 C CNN
+F 3 "http://ww1.microchip.com/downloads/en/DeviceDoc/25022B.pdf" H 2700 2450 50  0001 C CNN
+	1    2700 2450
+	1    0    0    -1
+$EndComp
+$Comp
+L Connector:Conn_01x14_Male J1
+U 1 1 5D145F9E
+P 1600 2550
+F 0 "J1" H 1708 3331 50  0000 C CNN
+F 1 "Left" H 1708 3240 50  0000 C CNN
+F 2 "Connector_PinHeader_2.54mm:PinHeader_1x14_P2.54mm_Vertical" H 1600 2550 50  0001 C CNN
+F 3 "~" H 1600 2550 50  0001 C CNN
+	1    1600 2550
+	1    0    0    -1
+$EndComp
+Text Label 2200 3150 2    50   ~ 0
 A16
-Text Label 2300 3050 2    50   ~ 0
+Text Label 2200 3050 2    50   ~ 0
 A15
-Text Label 2300 2950 2    50   ~ 0
+Text Label 2200 2950 2    50   ~ 0
 A14
-Text Label 2300 2850 2    50   ~ 0
+Text Label 2200 2850 2    50   ~ 0
 A13
-Text Label 2300 2750 2    50   ~ 0
+Text Label 2200 2750 2    50   ~ 0
 A12
-Text Label 2300 2650 2    50   ~ 0
+Text Label 2200 2650 2    50   ~ 0
 A11
-Text Label 2300 2550 2    50   ~ 0
+Text Label 2200 2550 2    50   ~ 0
 A10
-Text Label 2300 2450 2    50   ~ 0
+Text Label 2200 2450 2    50   ~ 0
 A9
-Text Label 2300 2350 2    50   ~ 0
+Text Label 2200 2350 2    50   ~ 0
 A8
-Text Label 2300 2250 2    50   ~ 0
+Text Label 2200 2250 2    50   ~ 0
 A7
-Text Label 2300 2150 2    50   ~ 0
+Text Label 2200 2150 2    50   ~ 0
 A6
-Text Label 2300 2050 2    50   ~ 0
+Text Label 2200 2050 2    50   ~ 0
 A5
-Text Label 2300 1950 2    50   ~ 0
+Text Label 2200 1950 2    50   ~ 0
 A4
-Text Label 2300 1850 2    50   ~ 0
+Text Label 2200 1850 2    50   ~ 0
 A3
-Text Label 2300 1750 2    50   ~ 0
+Text Label 2200 1750 2    50   ~ 0
 A2
-Text Label 3100 1750 0    50   ~ 0
+Text Label 3200 1750 0    50   ~ 0
 D0
-Text Label 3100 1850 0    50   ~ 0
+Text Label 3200 1850 0    50   ~ 0
 D1
-Text Label 3100 1950 0    50   ~ 0
+Text Label 3200 1950 0    50   ~ 0
 D2
-Text Label 3100 2050 0    50   ~ 0
+Text Label 3200 2050 0    50   ~ 0
 D3
-Text Label 3100 2150 0    50   ~ 0
+Text Label 3200 2150 0    50   ~ 0
 D4
-Text Label 3100 2250 0    50   ~ 0
+Text Label 3200 2250 0    50   ~ 0
 D5
-Text Label 3100 2350 0    50   ~ 0
+Text Label 3200 2350 0    50   ~ 0
 D6
-Text Label 3100 2450 0    50   ~ 0
+Text Label 3200 2450 0    50   ~ 0
 D7
-Text Label 3100 2850 0    50   ~ 0
+Text Label 3200 2850 0    50   ~ 0
 ~CS~
 $Comp
 L power:+5V #PWR0101
 U 1 1 5D154CE6
-P 3100 1550
-F 0 "#PWR0101" H 3100 1400 50  0001 C CNN
-F 1 "+5V" H 3100 1700 50  0000 C CNN
-F 2 "" H 3100 1550 50  0001 C CNN
-F 3 "" H 3100 1550 50  0001 C CNN
-	1    3100 1550
+P 3200 1550
+F 0 "#PWR0101" H 3200 1400 50  0001 C CNN
+F 1 "+5V" H 3200 1700 50  0000 C CNN
+F 2 "" H 3200 1550 50  0001 C CNN
+F 3 "" H 3200 1550 50  0001 C CNN
+	1    3200 1550
 	1    0    0    -1
 $EndComp
@@
 L power:GND #PWR0103
 U 1 1 5D155DE4
-P 3100 3550
-F 0 "#PWR0103" H 3100 3300 50  0001 C CNN
-F 1 "GND" H 3100 3400 50  0000 C CNN
-F 2 "" H 3100 3550 50  0001 C CNN
-F 3 "" H 3100 3550 50  0001 C CNN
-	1    3100 3550
-	1    0    0    -1
-$EndComp
-Text Label 2300 1550 2    50   ~ 0
+P 3200 3550
+F 0 "#PWR0103" H 3200 3300 50  0001 C CNN
+F 1 "GND" H 3200 3400 50  0000 C CNN
+F 2 "" H 3200 3550 50  0001 C CNN
+F 3 "" H 3200 3550 50  0001 C CNN
+	1    3200 3550
+	1    0    0    -1
+$EndComp
+Text Label 1800 1950 0    50   ~ 0
+A15
+Text Label 1800 2050 0    50   ~ 0
+A12
+Text Label 1800 2150 0    50   ~ 0
+A7
+Text Label 1800 2250 0    50   ~ 0
+A6
+Text Label 1800 2350 0    50   ~ 0
+A5
+Text Label 1800 2450 0    50   ~ 0
+A4
+Text Label 1800 2550 0    50   ~ 0
+A3
+Text Label 1800 2650 0    50   ~ 0
+A2
+Text Label 1800 2850 0    50   ~ 0
 A0
-Text Label 2300 1650 2    50   ~ 0
+Text Label 1800 2750 0    50   ~ 0
 A1
-Wire Wire Line
-	3100 3550 3100 3350
+Text Label 2200 1550 2    50   ~ 0
+A0
+Text Label 2200 1650 2    50   ~ 0
+A1
+Text Label 1800 2950 0    50   ~ 0
+D0
+Text Label 1800 3050 0    50   ~ 0
+D1
+Wire Wire Line
+	2200 3250 2200 3350
+Wire Wire Line
+	3200 3550 3200 3350
+Wire Wire Line
+	2200 3350 2200 3550
+Connection ~ 2200 3350
+Wire Wire Line
+	2200 3550 3200 3550
+Connection ~ 3200 3550
+Text Label 1800 3150 0    50   ~ 0
+D2
+$Comp
+L power:GND #PWR0104
+U 1 1 5D15888C
+P 1800 3250
+F 0 "#PWR0104" H 1800 3000 50  0001 C CNN
+F 1 "GND" H 1800 3100 50  0000 C CNN
+F 2 "" H 1800 3250 50  0001 C CNN
+F 3 "" H 1800 3250 50  0001 C CNN
+	1    1800 3250
+	1    0    0    -1
+$EndComp
+$Comp
+L Connector:Conn_01x14_Male J2
+U 1 1 5D162C4F
+P 3900 2550
+F 0 "J2" H 3872 2524 50  0000 R CNN
+F 1 "Right" H 3872 2433 50  0000 R CNN
+F 2 "Connector_PinHeader_2.54mm:PinHeader_1x14_P2.54mm_Vertical" H 3900 2550 50  0001 C CNN
+F 3 "~" H 3900 2550 50  0001 C CNN
+	1    3900 2550
+	-1   0    0    -1
+$EndComp
+$Comp
+L power:+5V #PWR0105
+U 1 1 5D1632D7
+P 3700 1950
+F 0 "#PWR0105" H 3700 1800 50  0001 C CNN
+F 1 "+5V" H 3700 2100 50  0000 C CNN
+F 2 "" H 3700 1950 50  0001 C CNN
+F 3 "" H 3700 1950 50  0001 C CNN
+	1    3700 1950
+	1    0    0    -1
+$EndComp
+Text Label 3700 2050 2    50   ~ 0
+A14
+Text Label 3700 2150 2    50   ~ 0
+A13
+Text Label 3700 2250 2    50   ~ 0
+A8
+Text Label 3700 2350 2    50   ~ 0
+A9
+Text Label 3700 2450 2    50   ~ 0
+A11
+Text Label 3700 2550 2    50   ~ 0
+A16
+Text Label 3700 2650 2    50   ~ 0
+A10
+Text Label 3700 2750 2    50   ~ 0
+~CS~
+Text Label 3700 2850 2    50   ~ 0
+D7
+Text Label 3700 2950 2    50   ~ 0
+D6
+Text Label 3700 3050 2    50   ~ 0
+D5
+Text Label 3700 3150 2    50   ~ 0
+D4
+Text Label 3700 3250 2    50   ~ 0
+D3
 $Comp
 L Device:R_Small R2
@@
 	1    0    0    -1
 $EndComp
-Text Label 3100 2950 0    50   ~ 0
+Text Label 3200 2950 0    50   ~ 0
 ~WE~
-Text Label 3100 3050 0    50   ~ 0
+Text Label 3200 3050 0    50   ~ 0
 ~OE~
 Text Label 4450 2500 0    50   ~ 0
@@
 	1    0    0    -1
 $EndComp
-$Comp
-L GW_RAM:Flash-512Kx8-PLCC-32 U1
-U 1 1 5E56BC07
-P 2700 2450
-F 0 "U1" H 2700 3500 50  0000 C CNN
-F 1 "39SF010" V 2700 2450 50  0000 C CNN
-F 2 "stdpads:PLCC-32" H 2700 2450 50  0001 C CNN
-F 3 "http://ww1.microchip.com/downloads/en/DeviceDoc/25022B.pdf" H 2700 2450 50  0001 C CNN
-	1    2700 2450
-	1    0    0    -1
-$EndComp
-Wire Wire Line
-	2300 3250 2300 3350
-Connection ~ 2300 3350
-Wire Wire Line
-	2300 3350 2300 3550
-Wire Wire Line
-	2300 3550 3100 3550
-Connection ~ 3100 3550
-$Comp
-L Connector_Generic:Conn_02x14_Counter_Clockwise J1
-U 1 1 5DECC3CD
-P 2200 4950
-F 0 "J1" H 2250 5767 50  0000 C CNN
-F 1 "Socket" H 2250 5676 50  0000 C CNN
-F 2 "stdpads:DIP-28_W15.24mm_Socket_Inverse_Forked" H 2200 4950 50  0001 C CNN
-F 3 "~" H 2200 4950 50  0001 C CNN
-	1    2200 4950
-	1    0    0    -1
-$EndComp
-Text Label 2000 4350 2    50   ~ 0
-A15
-Text Label 2000 4450 2    50   ~ 0
-A12
-Text Label 2000 4550 2    50   ~ 0
-A7
-Text Label 2000 4650 2    50   ~ 0
-A6
-Text Label 2000 4750 2    50   ~ 0
-A5
-Text Label 2000 4850 2    50   ~ 0
-A4
-Text Label 2000 4950 2    50   ~ 0
-A3
-Text Label 2000 5050 2    50   ~ 0
-A2
-Text Label 2000 5250 2    50   ~ 0
-A0
-Text Label 2000 5150 2    50   ~ 0
-A1
-Text Label 2000 5350 2    50   ~ 0
-D0
-Text Label 2000 5450 2    50   ~ 0
-D1
-Text Label 2000 5550 2    50   ~ 0
-D2
-$Comp
-L power:GND #PWR0104
-U 1 1 5DED018D
-P 2000 5650
-F 0 "#PWR0104" H 2000 5400 50  0001 C CNN
-F 1 "GND" H 2000 5500 50  0000 C CNN
-F 2 "" H 2000 5650 50  0001 C CNN
-F 3 "" H 2000 5650 50  0001 C CNN
-	1    2000 5650
-	1    0    0    -1
-$EndComp
-Text Label 2500 4450 0    50   ~ 0
-A14
-Text Label 2500 4550 0    50   ~ 0
-A13
-Text Label 2500 4650 0    50   ~ 0
-A8
-Text Label 2500 4750 0    50   ~ 0
-A9
-Text Label 2500 4850 0    50   ~ 0
-A11
-Text Label 2500 4950 0    50   ~ 0
-A16
-Text Label 2500 5050 0    50   ~ 0
-A10
-Text Label 2500 5150 0    50   ~ 0
-~CS~
-Text Label 2500 5250 0    50   ~ 0
-D7
-Text Label 2500 5350 0    50   ~ 0
-D6
-Text Label 2500 5450 0    50   ~ 0
-D5
-Text Label 2500 5550 0    50   ~ 0
-D4
-Text Label 2500 5650 0    50   ~ 0
-D3
-$Comp
-L power:+5V #PWR0105
-U 1 1 5DED0AF5
-P 2500 4350
-F 0 "#PWR0105" H 2500 4200 50  0001 C CNN
-F 1 "+5V" H 2500 4500 50  0000 C CNN
-F 2 "" H 2500 4350 50  0001 C CNN
-F 3 "" H 2500 4350 50  0001 C CNN
-	1    2500 4350
-	1    0    0    -1
-$EndComp

Commit message: Forked header, as submitted to JLCPCB
Parts:
- removed J1: Left, Connector_PinHeader_2.54mm:PinHeader_1x14_P2.54mm_Vertical, symbol Connector:Conn_01x14_Male
- removed J2: Right, Connector_PinHeader_2.54mm:PinHeader_1x14_P2.54mm_Vertical, symbol Connector:Conn_01x14_Male
- added J1: Socket, stdpads:DIP-28_W15.24mm_Socket_Inverse_Forked, symbol Connector_Generic:Conn_02x14_Counter_Clockwise
- U1: symbol stdparts:39F040 -> GW_RAM:Flash-512Kx8-PLCC-32
Connections:
- net +5V: now also J1.28 (Pin_28)
- net A0: now also J1.10 (Pin_10)
- net A1: now also J1.9 (Pin_9)
- net A10: now also J1.21 (Pin_21)
- net A11: now also J1.23 (Pin_23)
- net A12: now also J1.2 (Pin_2)
- net A13: now also J1.26 (Pin_26)
- net A14: now also J1.27 (Pin_27)
- net A15: now also J1.1 (Pin_1)
- net A16: now also J1.22 (Pin_22)
- net A2: now also J1.8 (Pin_8)
- net A3: now also J1.7 (Pin_7)
- net A4: now also J1.6 (Pin_6)
- net A5: now also J1.5 (Pin_5)
- net A6: now also J1.4 (Pin_4)
- net A7: now also J1.3 (Pin_3)
- net A8: now also J1.25 (Pin_25)
- net A9: now also J1.24 (Pin_24)
- net D0: now also J1.11 (Pin_11)
- net D1: now also J1.12 (Pin_12)
- net D2: now also J1.13 (Pin_13)
- net D3: now also J1.15 (Pin_15)
- net D4: now also J1.16 (Pin_16)
- net D5: now also J1.17 (Pin_17)
- net D6: now also J1.18 (Pin_18)
- net D7: now also J1.19 (Pin_19)
- net GND: now also J1.14 (Pin_14)
- net ~CS~: now also J1.20 (Pin_20)
Changed lines of the file:
@@
 	1    0    0    -1
 $EndComp
-$Comp
-L stdparts:39F040 U1
-U 1 1 5E56BC07
-P 2700 2450
-F 0 "U1" H 2700 3500 50  0000 C CNN
-F 1 "39SF010" V 2700 2450 50  0000 C CNN
-F 2 "stdpads:PLCC-32" H 2700 2450 50  0001 C CNN
-F 3 "http://ww1.microchip.com/downloads/en/DeviceDoc/25022B.pdf" H 2700 2450 50  0001 C CNN
-	1    2700 2450
-	1    0    0    -1
-$EndComp
-$Comp
-L Connector:Conn_01x14_Male J1
-U 1 1 5D145F9E
-P 1600 2550
-F 0 "J1" H 1708 3331 50  0000 C CNN
-F 1 "Left" H 1708 3240 50  0000 C CNN
-F 2 "Connector_PinHeader_2.54mm:PinHeader_1x14_P2.54mm_Vertical" H 1600 2550 50  0001 C CNN
-F 3 "~" H 1600 2550 50  0001 C CNN
-	1    1600 2550
-	1    0    0    -1
-$EndComp
-Text Label 2200 3150 2    50   ~ 0
+Text Label 2300 3150 2    50   ~ 0
 A16
-Text Label 2200 3050 2    50   ~ 0
+Text Label 2300 3050 2    50   ~ 0
 A15
-Text Label 2200 2950 2    50   ~ 0
+Text Label 2300 2950 2    50   ~ 0
 A14
-Text Label 2200 2850 2    50   ~ 0
+Text Label 2300 2850 2    50   ~ 0
 A13
-Text Label 2200 2750 2    50   ~ 0
+Text Label 2300 2750 2    50   ~ 0
 A12
-Text Label 2200 2650 2    50   ~ 0
+Text Label 2300 2650 2    50   ~ 0
 A11
-Text Label 2200 2550 2    50   ~ 0
+Text Label 2300 2550 2    50   ~ 0
 A10
-Text Label 2200 2450 2    50   ~ 0
+Text Label 2300 2450 2    50   ~ 0
 A9
-Text Label 2200 2350 2    50   ~ 0
+Text Label 2300 2350 2    50   ~ 0
 A8
-Text Label 2200 2250 2    50   ~ 0
+Text Label 2300 2250 2    50   ~ 0
 A7
-Text Label 2200 2150 2    50   ~ 0
+Text Label 2300 2150 2    50   ~ 0
 A6
-Text Label 2200 2050 2    50   ~ 0
+Text Label 2300 2050 2    50   ~ 0
 A5
-Text Label 2200 1950 2    50   ~ 0
+Text Label 2300 1950 2    50   ~ 0
 A4
-Text Label 2200 1850 2    50   ~ 0
+Text Label 2300 1850 2    50   ~ 0
 A3
-Text Label 2200 1750 2    50   ~ 0
+Text Label 2300 1750 2    50   ~ 0
 A2
-Text Label 3200 1750 0    50   ~ 0
+Text Label 3100 1750 0    50   ~ 0
 D0
-Text Label 3200 1850 0    50   ~ 0
+Text Label 3100 1850 0    50   ~ 0
 D1
-Text Label 3200 1950 0    50   ~ 0
+Text Label 3100 1950 0    50   ~ 0
 D2
-Text Label 3200 2050 0    50   ~ 0
+Text Label 3100 2050 0    50   ~ 0
 D3
-Text Label 3200 2150 0    50   ~ 0
+Text Label 3100 2150 0    50   ~ 0
 D4
-Text Label 3200 2250 0    50   ~ 0
+Text Label 3100 2250 0    50   ~ 0
 D5
-Text Label 3200 2350 0    50   ~ 0
+Text Label 3100 2350 0    50   ~ 0
 D6
-Text Label 3200 2450 0    50   ~ 0
+Text Label 3100 2450 0    50   ~ 0
 D7
-Text Label 3200 2850 0    50   ~ 0
+Text Label 3100 2850 0    50   ~ 0
 ~CS~
 $Comp
 L power:+5V #PWR0101
 U 1 1 5D154CE6
-P 3200 1550
-F 0 "#PWR0101" H 3200 1400 50  0001 C CNN
-F 1 "+5V" H 3200 1700 50  0000 C CNN
-F 2 "" H 3200 1550 50  0001 C CNN
-F 3 "" H 3200 1550 50  0001 C CNN
-	1    3200 1550
+P 3100 1550
+F 0 "#PWR0101" H 3100 1400 50  0001 C CNN
+F 1 "+5V" H 3100 1700 50  0000 C CNN
+F 2 "" H 3100 1550 50  0001 C CNN
+F 3 "" H 3100 1550 50  0001 C CNN
+	1    3100 1550
 	1    0    0    -1
 $EndComp
@@
 L power:GND #PWR0103
 U 1 1 5D155DE4
-P 3200 3550
-F 0 "#PWR0103" H 3200 3300 50  0001 C CNN
-F 1 "GND" H 3200 3400 50  0000 C CNN
-F 2 "" H 3200 3550 50  0001 C CNN
-F 3 "" H 3200 3550 50  0001 C CNN
-	1    3200 3550
-	1    0    0    -1
-$EndComp
-Text Label 1800 1950 0    50   ~ 0
-A15
-Text Label 1800 2050 0    50   ~ 0
-A12
-Text Label 1800 2150 0    50   ~ 0
-A7
-Text Label 1800 2250 0    50   ~ 0
-A6
-Text Label 1800 2350 0    50   ~ 0
-A5
-Text Label 1800 2450 0    50   ~ 0
-A4
-Text Label 1800 2550 0    50   ~ 0
-A3
-Text Label 1800 2650 0    50   ~ 0
-A2
-Text Label 1800 2850 0    50   ~ 0
+P 3100 3550
+F 0 "#PWR0103" H 3100 3300 50  0001 C CNN
+F 1 "GND" H 3100 3400 50  0000 C CNN
+F 2 "" H 3100 3550 50  0001 C CNN
+F 3 "" H 3100 3550 50  0001 C CNN
+	1    3100 3550
+	1    0    0    -1
+$EndComp
+Text Label 2300 1550 2    50   ~ 0
 A0
-Text Label 1800 2750 0    50   ~ 0
+Text Label 2300 1650 2    50   ~ 0
 A1
-Text Label 2200 1550 2    50   ~ 0
-A0
-Text Label 2200 1650 2    50   ~ 0
-A1
-Text Label 1800 2950 0    50   ~ 0
-D0
-Text Label 1800 3050 0    50   ~ 0
-D1
-Wire Wire Line
-	2200 3250 2200 3350
-Wire Wire Line
-	3200 3550 3200 3350
-Wire Wire Line
-	2200 3350 2200 3550
-Connection ~ 2200 3350
-Wire Wire Line
-	2200 3550 3200 3550
-Connection ~ 3200 3550
-Text Label 1800 3150 0    50   ~ 0
-D2
-$Comp
-L power:GND #PWR0104
-U 1 1 5D15888C
-P 1800 3250
-F 0 "#PWR0104" H 1800 3000 50  0001 C CNN
-F 1 "GND" H 1800 3100 50  0000 C CNN
-F 2 "" H 1800 3250 50  0001 C CNN
-F 3 "" H 1800 3250 50  0001 C CNN
-	1    1800 3250
-	1    0    0    -1
-$EndComp
-$Comp
-L Connector:Conn_01x14_Male J2
-U 1 1 5D162C4F
-P 3900 2550
-F 0 "J2" H 3872 2524 50  0000 R CNN
-F 1 "Right" H 3872 2433 50  0000 R CNN
-F 2 "Connector_PinHeader_2.54mm:PinHeader_1x14_P2.54mm_Vertical" H 3900 2550 50  0001 C CNN
-F 3 "~" H 3900 2550 50  0001 C CNN
-	1    3900 2550
-	-1   0    0    -1
-$EndComp
-$Comp
-L power:+5V #PWR0105
-U 1 1 5D1632D7
-P 3700 1950
-F 0 "#PWR0105" H 3700 1800 50  0001 C CNN
-F 1 "+5V" H 3700 2100 50  0000 C CNN
-F 2 "" H 3700 1950 50  0001 C CNN
-F 3 "" H 3700 1950 50  0001 C CNN
-	1    3700 1950
-	1    0    0    -1
-$EndComp
-Text Label 3700 2050 2    50   ~ 0
-A14
-Text Label 3700 2150 2    50   ~ 0
-A13
-Text Label 3700 2250 2    50   ~ 0
-A8
-Text Label 3700 2350 2    50   ~ 0
-A9
-Text Label 3700 2450 2    50   ~ 0
-A11
-Text Label 3700 2550 2    50   ~ 0
-A16
-Text Label 3700 2650 2    50   ~ 0
-A10
-Text Label 3700 2750 2    50   ~ 0
-~CS~
-Text Label 3700 2850 2    50   ~ 0
-D7
-Text Label 3700 2950 2    50   ~ 0
-D6
-Text Label 3700 3050 2    50   ~ 0
-D5
-Text Label 3700 3150 2    50   ~ 0
-D4
-Text Label 3700 3250 2    50   ~ 0
-D3
+Wire Wire Line
+	3100 3550 3100 3350
 $Comp
 L Device:R_Small R2
@@
 	1    0    0    -1
 $EndComp
-Text Label 3200 2950 0    50   ~ 0
+Text Label 3100 2950 0    50   ~ 0
 ~WE~
-Text Label 3200 3050 0    50   ~ 0
+Text Label 3100 3050 0    50   ~ 0
 ~OE~
 Text Label 4450 2500 0    50   ~ 0
@@
 	1    0    0    -1
 $EndComp
+$Comp
+L GW_RAM:Flash-512Kx8-PLCC-32 U1
+U 1 1 5E56BC07
+P 2700 2450
+F 0 "U1" H 2700 3500 50  0000 C CNN
+F 1 "39SF010" V 2700 2450 50  0000 C CNN
+F 2 "stdpads:PLCC-32" H 2700 2450 50  0001 C CNN
+F 3 "http://ww1.microchip.com/downloads/en/DeviceDoc/25022B.pdf" H 2700 2450 50  0001 C CNN
+	1    2700 2450
+	1    0    0    -1
+$EndComp
+Wire Wire Line
+	2300 3250 2300 3350
+Connection ~ 2300 3350
+Wire Wire Line
+	2300 3350 2300 3550
+Wire Wire Line
+	2300 3550 3100 3550
+Connection ~ 3100 3550
+$Comp
+L Connector_Generic:Conn_02x14_Counter_Clockwise J1
+U 1 1 5DECC3CD
+P 2200 4950
+F 0 "J1" H 2250 5767 50  0000 C CNN
+F 1 "Socket" H 2250 5676 50  0000 C CNN
+F 2 "stdpads:DIP-28_W15.24mm_Socket_Inverse_Forked" H 2200 4950 50  0001 C CNN
+F 3 "~" H 2200 4950 50  0001 C CNN
+	1    2200 4950
+	1    0    0    -1
+$EndComp
+Text Label 2000 4350 2    50   ~ 0
+A15
+Text Label 2000 4450 2    50   ~ 0
+A12
+Text Label 2000 4550 2    50   ~ 0
+A7
+Text Label 2000 4650 2    50   ~ 0
+A6
+Text Label 2000 4750 2    50   ~ 0
+A5
+Text Label 2000 4850 2    50   ~ 0
+A4
+Text Label 2000 4950 2    50   ~ 0
+A3
+Text Label 2000 5050 2    50   ~ 0
+A2
+Text Label 2000 5250 2    50   ~ 0
+A0
+Text Label 2000 5150 2    50   ~ 0
+A1
+Text Label 2000 5350 2    50   ~ 0
+D0
+Text Label 2000 5450 2    50   ~ 0
+D1
+Text Label 2000 5550 2    50   ~ 0
+D2
+$Comp
+L power:GND #PWR0104
+U 1 1 5DED018D
+P 2000 5650
+F 0 "#PWR0104" H 2000 5400 50  0001 C CNN
+F 1 "GND" H 2000 5500 50  0000 C CNN
+F 2 "" H 2000 5650 50  0001 C CNN
+F 3 "" H 2000 5650 50  0001 C CNN
+	1    2000 5650
+	1    0    0    -1
+$EndComp
+Text Label 2500 4450 0    50   ~ 0
+A14
+Text Label 2500 4550 0    50   ~ 0
+A13
+Text Label 2500 4650 0    50   ~ 0
+A8
+Text Label 2500 4750 0    50   ~ 0
+A9
+Text Label 2500 4850 0    50   ~ 0
+A11
+Text Label 2500 4950 0    50   ~ 0
+A16
+Text Label 2500 5050 0    50   ~ 0
+A10
+Text Label 2500 5150 0    50   ~ 0
+~CS~
+Text Label 2500 5250 0    50   ~ 0
+D7
+Text Label 2500 5350 0    50   ~ 0
+D6
+Text Label 2500 5450 0    50   ~ 0
+D5
+Text Label 2500 5550 0    50   ~ 0
+D4
+Text Label 2500 5650 0    50   ~ 0
+D3
+$Comp
+L power:+5V #PWR0105
+U 1 1 5DED0AF5
+P 2500 4350
+F 0 "#PWR0105" H 2500 4200 50  0001 C CNN
+F 1 "+5V" H 2500 4500 50  0000 C CNN
+F 2 "" H 2500 4350 50  0001 C CNN
+F 3 "" H 2500 4350 50  0001 C CNN
+	1    2500 4350
+	1    0    0    -1
+$EndComp
