File: GW28R8128.sch (KiCad schematic (older format))
At the start: 8 parts, among them J1 Socket, U1 39SF010

Commit message: Revised
Parts:
- added FID4: Fiducial, stdpads:Fiducial, symbol Mechanical:Fiducial
- added TP1: ~OE~, stdpads:Tyco_RCU_0603_Paste, symbol Connector:TestPoint
- added TP2: ~WE~, stdpads:Tyco_RCU_0603_Paste, symbol Connector:TestPoint
- C1: value 100n -> 10u
Connections:
- net ~OE~: now also TP1.1
- net ~WE~: now also TP2.1
Other:
- moved on the sheet: R1, R2
Changed lines of the file:
@@
 EESchema Schematic File Version 4
-LIBS:GW28R8128-cache
-EELAYER 29 0
+EELAYER 30 0
 EELAYER END
 $Descr USLetter 11000 8500
@@
 P 4450 1850
 F 0 "C1" H 4500 1900 50  0000 L CNN
-F 1 "100n" H 4500 1800 50  0000 L CNN
+F 1 "10u" H 4500 1800 50  0000 L CNN
 F 2 "stdpads:C_0805" H 4450 1850 50  0001 C CNN
 F 3 "~" H 4450 1850 50  0001 C CNN
@@
 Wire Wire Line
 	3100 3550 3100 3350
-$Comp
-L Device:R_Small R2
-U 1 1 5D31EA5F
-P 4850 2600
-F 0 "R2" H 4909 2646 50  0000 L CNN
-F 1 "22k" H 4909 2555 50  0000 L CNN
-F 2 "stdpads:R_0805" H 4850 2600 50  0001 C CNN
-F 3 "~" H 4850 2600 50  0001 C CNN
-	1    4850 2600
-	1    0    0    -1
-$EndComp
-$Comp
-L power:+5V #PWR0102
-U 1 1 5D31EC78
-P 4850 2500
-F 0 "#PWR0102" H 4850 2350 50  0001 C CNN
-F 1 "+5V" H 4850 2650 50  0000 C CNN
-F 2 "" H 4850 2500 50  0001 C CNN
-F 3 "" H 4850 2500 50  0001 C CNN
-	1    4850 2500
-	1    0    0    -1
-$EndComp
 Text Label 3100 2950 0    50   ~ 0
 ~WE~
 Text Label 3100 3050 0    50   ~ 0
 ~OE~
-Text Label 4450 2500 0    50   ~ 0
+Text Label 5650 2500 0    50   ~ 0
 ~OE~
 $Comp
 L Device:R_Small R1
 U 1 1 5D3208E4
-P 4450 2600
-F 0 "R1" H 4509 2646 50  0000 L CNN
-F 1 "22k" H 4509 2555 50  0000 L CNN
-F 2 "stdpads:R_0805" H 4450 2600 50  0001 C CNN
-F 3 "~" H 4450 2600 50  0001 C CNN
-	1    4450 2600
+P 5650 2600
+F 0 "R1" H 5709 2646 50  0000 L CNN
+F 1 "22k" H 5709 2555 50  0000 L CNN
+F 2 "stdpads:R_0805" H 5650 2600 50  0001 C CNN
+F 3 "~" H 5650 2600 50  0001 C CNN
+	1    5650 2600
 	1    0    0    -1
 $EndComp
@@
 L power:GND #PWR0106
 U 1 1 5D3208EA
-P 4450 2700
-F 0 "#PWR0106" H 4450 2450 50  0001 C CNN
-F 1 "GND" H 4450 2550 50  0000 C CNN
-F 2 "" H 4450 2700 50  0001 C CNN
-F 3 "" H 4450 2700 50  0001 C CNN
-	1    4450 2700
-	1    0    0    -1
-$EndComp
-Text Label 4850 2800 2    50   ~ 0
-~WE~
-Wire Wire Line
-	4850 2800 4850 2700
+P 5650 2700
+F 0 "#PWR0106" H 5650 2450 50  0001 C CNN
+F 1 "GND" H 5650 2550 50  0000 C CNN
+F 2 "" H 5650 2700 50  0001 C CNN
+F 3 "" H 5650 2700 50  0001 C CNN
+	1    5650 2700
+	1    0    0    -1
+$EndComp
 $Comp
 L Mechanical:Fiducial FID1
@@
 	1    0    0    -1
 $EndComp
+$Comp
+L Device:R_Small R2
+U 1 1 5D31EA5F
+P 5050 2600
+F 0 "R2" H 5109 2646 50  0000 L CNN
+F 1 "22k" H 5109 2555 50  0000 L CNN
+F 2 "stdpads:R_0805" H 5050 2600 50  0001 C CNN
+F 3 "~" H 5050 2600 50  0001 C CNN
+	1    5050 2600
+	1    0    0    -1
+$EndComp
+$Comp
+L power:+5V #PWR0102
+U 1 1 5D31EC78
+P 5050 2500
+F 0 "#PWR0102" H 5050 2350 50  0001 C CNN
+F 1 "+5V" H 5050 2650 50  0000 C CNN
+F 2 "" H 5050 2500 50  0001 C CNN
+F 3 "" H 5050 2500 50  0001 C CNN
+	1    5050 2500
+	1    0    0    -1
+$EndComp
+Text Label 5050 2800 2    50   ~ 0
+~WE~
+Wire Wire Line
+	5050 2800 5050 2700
+$Comp
+L Connector:TestPoint TP1
+U 1 1 5EC596B7
+P 5350 2500
+F 0 "TP1" H 5408 2624 50  0000 L CNN
+F 1 "~OE~" H 5408 2526 50  0000 L CNN
+F 2 "stdpads:Tyco_RCU_0603_Paste" H 5550 2500 50  0001 C CNN
+F 3 "~" H 5550 2500 50  0001 C CNN
+	1    5350 2500
+	1    0    0    -1
+$EndComp
+$Comp
+L Connector:TestPoint TP2
+U 1 1 5EC59B6C
+P 5350 2800
+F 0 "TP2" H 5408 2924 50  0000 L CNN
+F 1 "~WE~" H 5408 2826 50  0000 L CNN
+F 2 "stdpads:Tyco_RCU_0603_Paste" H 5550 2800 50  0001 C CNN
+F 3 "~" H 5550 2800 50  0001 C CNN
+	1    5350 2800
+	1    0    0    -1
+$EndComp
+Wire Wire Line
+	5350 2800 5050 2800
+Wire Wire Line
+	5650 2500 5350 2500
+$Comp
+L Mechanical:Fiducial FID4
+U 1 1 5EC61517
+P 4500 4050
+F 0 "FID4" H 4585 4096 50  0000 L CNN
+F 1 "Fiducial" H 4585 4005 50  0000 L CNN
+F 2 "stdpads:Fiducial" H 4500 4050 50  0001 C CNN
+F 3 "~" H 4500 4050 50  0001 C CNN
+	1    4500 4050
+	1    0    0    -1
+$EndComp

Commit message: Small update
Parts:
- C1: value 10u -> 2u2
Changed lines of the file:
@@
 P 4450 1850
 F 0 "C1" H 4500 1900 50  0000 L CNN
-F 1 "10u" H 4500 1800 50  0000 L CNN
+F 1 "2u2" H 4500 1800 50  0000 L CNN
 F 2 "stdpads:C_0805" H 4450 1850 50  0001 C CNN
 F 3 "~" H 4450 1850 50  0001 C CNN
