File: GW28R8128.kicad_sch (KiCad schematic)
At the start: 11 parts, among them J1 Socket, U1 39SF010

Commit message: New with fuse
Parts:
- removed FID1, FID2, FID3, FID4: Fiducial, stdpads:Fiducial, symbol Mechanical:Fiducial
- added C1: 2u2, stdpads:C_0805, symbol Device:C_Small
- added D1: B340B, stdpads:D_SMB, symbol Device:D_Schottky_Small_Filled
- added F1: 200mA, stdpads:BelFuse_1210, symbol Device:Polyfuse_Small
- TP1: value ~OE~ -> ~{OE}
- TP2: value ~WE~ -> ~{WE}
- renumbered C1 to C2
Connections:
- net +5V: now also D1.1 (K), F1.2; no longer J1.28 (Pin_28)
- net GND: now also C1.2, D1.2 (A)
- new net VCC: C1.1, F1.1, J1.28 (Pin_28)
Other:
- moved on the sheet: C2, TP1, TP2
